File: _autosave-DINODE.sch (KiCad schematic (older format))
At the start: 32 parts, among them J1 Barrel_Jack, J10 Conn_01x03_Male, J11 Conn_02x04_Odd_Even, J12 Conn_01x03_Female, J13 Conn_02x04_Odd_Even, J2 Conn_01x02_Male, J3 Conn_01x07, J4 Conn_01x16, J5 Conn_02x04_Odd_Even, J6 Conn_02x04_Odd_Even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

Commit message: Started routing
Connections:
- net +12V: now reaches C3.1, C5.1, J1.1, U1.1 (IN)
Changed lines of the file:
@@
 	650  1200 650  850
 Wire Wire Line
-	650  850  1000 850
+	650  850  800  850
 Wire Wire Line
 	1000 850  1250 850
@@
 Wire Notes Line
 	550  500  550  1750
+$Comp
+L power:+12V #PWR0105
+U 1 1 5DEF303B
+P 800 750
+F 0 "#PWR0105" H 800 600 50  0001 C CNN
+F 1 "+12V" H 815 923 50  0000 C CNN
+F 2 "" H 800 750 50  0001 C CNN
+F 3 "" H 800 750 50  0001 C CNN
+	1    800  750
+	1    0    0    -1
+$EndComp
+Wire Wire Line
+	800  750  800  850
+Connection ~ 800  850
+Wire Wire Line
+	800  850  1000 850
 $EndSCHEMATC
