File: DINODE.sch (KiCad schematic (older format))
At the start: 35 parts, among them J1 Barrel_Jack, J10 Conn_01x03_Male, J11 Conn_02x04_Odd_Even, J12 Conn_01x03_Female, J13 Conn_02x04_Odd_Even, J2 Conn_01x02_Male, J3 Conn_01x07, J4 Conn_01x16, J5 Conn_02x04_Odd_Even, J6 Conn_02x04_Odd_Even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

Commit message: Added gerber files
Changed lines of the file:
@@
 	1    0    0    -1
 $EndComp
-Text Label 5850 2350 0    50   ~ 0
-ESP8266
 $EndSCHEMATC
