File: DINODE.sch (KiCad schematic (older format))
At the start: 32 parts, among them J1 Barrel_Jack, J10 Conn_01x03_Male, J11 Conn_02x04_Odd_Even, J12 Conn_01x03_Female, J13 Conn_02x04_Odd_Even, J2 Conn_01x02_Male, J3 Conn_01x07, J4 Conn_01x16, J5 Conn_02x04_Odd_Even, J6 Conn_02x04_Odd_Even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

Commit message: Port C routing
Connections:
- net MISO: now also J9.7 (Pin_7), U2.2 (PB6)
- net MOSI: no longer J9.7 (Pin_7), U2.2 (PB6)
- net RESET: now also SW1.2, U2.4 (~RESET)
- net +12V: now reaches C3.1, C5.1, J1.1, U1.1 (IN)
Changed lines of the file:
@@
 MOSI
 Text GLabel 4400 4250 2    50   Input ~ 0
-MOSI
+MISO
 Text GLabel 3950 4350 2    50   Input ~ 0
 SCK
@@
 	650  1200 650  850
 Wire Wire Line
-	650  850  1000 850
+	650  850  800  850
 Wire Wire Line
 	1000 850  1250 850
@@
 Connection ~ 1000 1200
 Wire Wire Line
-	1850 2750 2150 2750
+	1850 2750 2050 2750
 Wire Wire Line
 	7650 950  7900 950
@@
 Wire Notes Line
 	550  500  550  1750
+$Comp
+L power:+12V #PWR0105
+U 1 1 5DEF303B
+P 800 750
+F 0 "#PWR0105" H 800 600 50  0001 C CNN
+F 1 "+12V" H 815 923 50  0000 C CNN
+F 2 "" H 800 750 50  0001 C CNN
+F 3 "" H 800 750 50  0001 C CNN
+	1    800  750
+	1    0    0    -1
+$EndComp
+Wire Wire Line
+	800  750  800  850
+Connection ~ 800  850
+Wire Wire Line
+	800  850  1000 850
+Text GLabel 2050 2650 1    50   Input ~ 0
+RESET
+Wire Wire Line
+	2050 2650 2050 2750
+Connection ~ 2050 2750
+Wire Wire Line
+	2050 2750 2150 2750
 $EndSCHEMATC

Commit message: Addition of edge cuts
Parts:
- added H1, H2, H3: MountingHole, MountingHole:MountingHole_3.2mm_M3, symbol Mechanical:MountingHole
Changed lines of the file:
@@
 Wire Wire Line
 	2050 2750 2150 2750
+$Comp
+L Mechanical:MountingHole H1
+U 1 1 5DECA203
+P 1500 7250
+F 0 "H1" H 1600 7296 50  0000 L CNN
+F 1 "MountingHole" H 1600 7205 50  0000 L CNN
+F 2 "MountingHole:MountingHole_3.2mm_M3" H 1500 7250 50  0001 C CNN
+F 3 "~" H 1500 7250 50  0001 C CNN
+	1    1500 7250
+	1    0    0    -1
+$EndComp
+$Comp
+L Mechanical:MountingHole H2
+U 1 1 5DECB2F7
+P 2250 7250
+F 0 "H2" H 2350 7296 50  0000 L CNN
+F 1 "MountingHole" H 2350 7205 50  0000 L CNN
+F 2 "MountingHole:MountingHole_3.2mm_M3" H 2250 7250 50  0001 C CNN
+F 3 "~" H 2250 7250 50  0001 C CNN
+	1    2250 7250
+	1    0    0    -1
+$EndComp
+$Comp
+L Mechanical:MountingHole H3
+U 1 1 5DECB7D9
+P 3100 7250
+F 0 "H3" H 3200 7296 50  0000 L CNN
+F 1 "MountingHole" H 3200 7205 50  0000 L CNN
+F 2 "MountingHole:MountingHole_3.2mm_M3" H 3100 7250 50  0001 C CNN
+F 3 "~" H 3100 7250 50  0001 C CNN
+	1    3100 7250
+	1    0    0    -1
+$EndComp
 $EndSCHEMATC

Commit message: updated gerber files
Connections:
- net PC_0: no longer J4.10 (Pin_10)
- net PC_1: no longer J4.9 (Pin_9)
- net PD_6: now also J4.10 (Pin_10)
- net PD_7: now also J4.9 (Pin_9)
Changed lines of the file:
@@
 PC_2
 Text GLabel 6300 4750 0    50   Input ~ 0
-PC_1
+PD_7
 Text GLabel 6300 4850 0    50   Input ~ 0
-PC_0
+PD_6
 Text GLabel 6300 4950 0    50   Input ~ 0
 PB_2
