File: _autosave-DINODE.kicad_pcb (KiCad board)
At the start: 2 copper layers, 74 x 90.2 mm, 36 parts, among them J1 Barrel_Jack, J10 Conn_01x03_Male, J11 Conn_02x04_Odd_Even, J12 Conn_01x03_Female, J13 Conn_02x04_Odd_Even, J2 Conn_01x02_Male, J3 Conn_01x07, J4 Conn_01x16, J5 Conn_02x04_Odd_Even, J6 Conn_02x04_Odd_Even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

Commit message: updated gerber files
Other:
- board text added: "jackagwaya@gmail.com"
Changed lines of the file:
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@@
   (general
     (thickness 1)
-    (drawings 73)
+    (drawings 74)
     (tracks 1034)
     (zones 0)
@@
     (pad 1 np_thru_hole circle (at 0 0) (size 3.2 3.2) (drill 3.2) (layers *.Cu *.Mask))
   )
+  (gr_text jackagwaya@gmail.com (at 121.412 86.106) (layer B.SilkS)
+    (effects (font (size 1 1) (thickness 0.15)) (justify mirror))
+  )
   (gr_circle (center 117.475 79.375) (end 117.602 79.121) (layer F.SilkS) (width 0.12))
   (gr_line (start 159.131 129.54) (end 130.81 129.54) (layer Edge.Cuts) (width 0.05))
@@
   (gr_line (start 159.131 45.72) (end 148.59 45.72) (layer Edge.Cuts) (width 0.05))
   (gr_line (start 159.131 60.198) (end 159.131 45.72) (layer Edge.Cuts) (width 0.05))
-  (gr_text "BY: JACK MCLEANS" (at 137.541 122.682) (layer B.SilkS)
+  (gr_text "BY: JACK MCLEANS" (at 122.809 83.947) (layer B.SilkS)
     (effects (font (size 1 1) (thickness 0.15)) (justify mirror))
   )
